File: Artemis Corner Board V2 FR.sch (EAGLE design)
At the start: 40 parts, among them U1 TPS562219, U10 TPS562219, U4 MCP2562FD

Commit message: Finally got shape right
Parts:
- added C72, C73: 10uF, adafruit:C-USC0805
- added JP8: (no value), pinhead:PINHD-1X2
- added LED6: GREEN, FormE:LEDCHIPLED_0805
- added R15: 0.007, adafruit:R-US_R0805
- added R18: 1K, adafruit:R-US_R0805
- added U21: LM1085IS, FormE:LM1085
Connections:
- new net +12V: JP8.1, LED6.A
- new net 12V_CURRENT_SENSE+: C73.1, R15.1, U21.OUT
- new net 12V_CURRENT_SENSE-: JP8.2, R15.2
- new net N$11: LED6.C, R18.2
- new net N$54: C72.1, U21.IN
- net GND: now also C72.2, C73.2, R18.1, U21.ADJ
Other:
- note added: "REGULATED OUTPUT"
Changed lines of the file:
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@@
 <part name="P+8" library="supply1" deviceset="VCC" device=""/>
 <part name="H2" library="FormE" deviceset="776228-4" device="" value="776228-4"/>
+<part name="GND9" library="supply1" deviceset="GND" device=""/>
+<part name="LED6" library="FormE" deviceset="LED" device="CHIPLED_0805" value="GREEN">
+<attribute name="PARTNO" value="598-8170-107F"/>
+</part>
+<part name="R18" library="adafruit" deviceset="R-US_" device="R0805" value="1K">
+<attribute name="PARTNO" value="ERJ-6ENF1001V"/>
+</part>
+<part name="GND24" library="supply1" deviceset="GND" device=""/>
+<part name="P+18" library="supply1" deviceset="+12V" device=""/>
+<part name="P+17" library="supply1" deviceset="+12V" device=""/>
+<part name="R15" library="adafruit" deviceset="R-US_" device="R0805" value="0.007">
+<attribute name="PARTNO" value="PMR10EZPFU7L00"/>
+</part>
+<part name="JP8" library="pinhead" deviceset="PINHD-1X2" device=""/>
+<part name="U21" library="FormE" deviceset="LM1085" device="" value="LM1085IS">
+<attribute name="PARTNO" value="LM1085IS-12/NOPB"/>
+</part>
+<part name="C72" library="adafruit" deviceset="C-US" device="C0805" value="10uF">
+<attribute name="PARTNO" value="GRM21BR61E106KA73L"/>
+</part>
+<part name="C73" library="adafruit" deviceset="C-US" device="C0805" value="10uF">
+<attribute name="PARTNO" value="GRM21BR61E106KA73L"/>
+</part>
 </parts>
 <sheets>
@@
 <text x="50.8" y="264.16" size="1.778" layer="95">LEDs that serve no practical function, exept to look "Sick as fuck"</text>
 <text x="129.54" y="340.36" size="6.223" layer="95" font="vector">ARTEMIS CORNER BOARD V2 FR</text>
+<text x="445.77" y="27.94" size="1.778" layer="91">REGULATED OUTPUT</text>
+<text x="422.91" y="-2.54" size="1.778" layer="91">25V or higher cap</text>
+<text x="342.9" y="-1.27" size="1.778" layer="91">25V or higher cap</text>
 </plain>
 <instances>
@@
 <instance part="P+8" gate="VCC" x="452.12" y="292.1"/>
 <instance part="H2" gate="G$2" x="474.98" y="254" rot="R180"/>
+<instance part="GND9" gate="1" x="394.97" y="-12.7"/>
+<instance part="LED6" gate="G$1" x="461.01" y="7.62">
+<attribute name="PARTNO" x="461.01" y="7.62" size="1.778" layer="96" display="off"/>
+</instance>
+<instance part="R18" gate="G$1" x="461.01" y="-5.08" rot="R90">
+<attribute name="PARTNO" x="461.01" y="-5.08" size="1.778" layer="96" display="off"/>
+</instance>
+<instance part="GND24" gate="1" x="461.01" y="-15.24"/>
+<instance part="P+18" gate="1" x="461.01" y="15.24"/>
+<instance part="P+17" gate="1" x="440.69" y="27.94"/>
+<instance part="R15" gate="G$1" x="430.53" y="10.16">
+<attribute name="PARTNO" x="430.53" y="10.16" size="1.778" layer="96" display="off"/>
+</instance>
+<instance part="JP8" gate="G$1" x="450.85" y="10.16"/>
+<instance part="U21" gate="G$1" x="392.43" y="5.08">
+<attribute name="PARTNO" x="392.43" y="5.08" size="1.778" layer="96" display="off"/>
+</instance>
+<instance part="C72" gate="G$1" x="374.65" y="5.08">
+<attribute name="PARTNO" x="374.65" y="5.08" size="1.778" layer="96" display="off"/>
+</instance>
+<instance part="C73" gate="G$1" x="415.29" y="5.08">
+<attribute name="PARTNO" x="415.29" y="5.08" size="1.778" layer="96" display="off"/>
+</instance>
 </instances>
 <busses>
@@
 <label x="454.66" y="281.94" size="1.778" layer="95"/>
 <pinref part="GND23" gate="1" pin="GND"/>
-<wire x1="459.74" y1="281.94" x2="449.58" y2="281.94" width="0.1524" layer="91"/>
+<wire x1="457.2" y1="281.94" x2="449.58" y2="281.94" width="0.1524" layer="91"/>
+</segment>
+<segment>
+<pinref part="GND24" gate="1" pin="GND"/>
+<pinref part="R18" gate="G$1" pin="1"/>
+<wire x1="461.01" y1="-12.7" x2="461.01" y2="-10.16" width="0.1524" layer="91"/>
+</segment>
+<segment>
+<pinref part="U21" gate="G$1" pin="ADJ"/>
+<pinref part="GND9" gate="1" pin="GND"/>
+<wire x1="394.97" y1="-2.54" x2="394.97" y2="-5.08" width="0.1524" layer="91"/>
+<pinref part="C72" gate="G$1" pin="2"/>
+<wire x1="394.97" y1="-5.08" x2="394.97" y2="-7.62" width="0.1524" layer="91"/>
+<wire x1="394.97" y1="-7.62" x2="394.97" y2="-10.16" width="0.1524" layer="91"/>
+<wire x1="374.65" y1="0" x2="374.65" y2="-5.08" width="0.1524" layer="91"/>
+<wire x1="374.65" y1="-5.08" x2="394.97" y2="-5.08" width="0.1524" layer="91"/>
+<junction x="394.97" y="-5.08"/>
+<pinref part="C73" gate="G$1" pin="2"/>
+<wire x1="415.29" y1="0" x2="415.29" y2="-7.62" width="0.1524" layer="91"/>
+<wire x1="415.29" y1="-7.62" x2="394.97" y2="-7.62" width="0.1524" layer="91"/>
+<junction x="394.97" y="-7.62"/>
 </segment>
 </net>
@@
 </segment>
 </net>
+<net name="+12V" class="0">
+<segment>
+<pinref part="P+18" gate="1" pin="+12V"/>
+<pinref part="LED6" gate="G$1" pin="A"/>
+<wire x1="461.01" y1="12.7" x2="461.01" y2="10.16" width="0.1524" layer="91"/>
+</segment>
+<segment>
+<pinref part="JP8" gate="G$1" pin="1"/>
+<pinref part="P+17" gate="1" pin="+12V"/>
+<wire x1="448.31" y1="12.7" x2="440.69" y2="12.7" width="0.1524" layer="91"/>
+<wire x1="440.69" y1="12.7" x2="440.69" y2="25.4" width="0.1524" layer="91"/>
+</segment>
+</net>
+<net name="N$11" class="0">
+<segment>
+<pinref part="R18" gate="G$1" pin="2"/>
+<pinref part="LED6" gate="G$1" pin="C"/>
+<wire x1="461.01" y1="0" x2="461.01" y2="2.54" width="0.1524" layer="91"/>
+</segment>
+</net>
+<net name="12V_CURRENT_SENSE+" class="0">
+<segment>
+<pinref part="R15" gate="G$1" pin="1"/>
+<pinref part="C73" gate="G$1" pin="1"/>
+<wire x1="415.29" y1="10.16" x2="425.45" y2="10.16" width="0.1524" layer="91"/>
+<wire x1="415.29" y1="7.62" x2="415.29" y2="10.16" width="0.1524" layer="91"/>
+<pinref part="U21" gate="G$1" pin="OUT"/>
+<wire x1="407.67" y1="10.16" x2="415.29" y2="10.16" width="0.1524" layer="91"/>
+<junction x="415.29" y="10.16"/>
+<label x="420.37" y="10.16" size="1.778" layer="95" rot="R90"/>
+</segment>
+</net>
+<net name="12V_CURRENT_SENSE-" class="0">
+<segment>
+<pinref part="R15" gate="G$1" pin="2"/>
+<wire x1="435.61" y1="10.16" x2="448.31" y2="10.16" width="0.1524" layer="91"/>
+<pinref part="JP8" gate="G$1" pin="2"/>
+<label x="435.61" y="10.16" size="1.778" layer="95" rot="R90"/>
+</segment>
+</net>
+<net name="N$54" class="0">
+<segment>
+<pinref part="U21" gate="G$1" pin="IN"/>
+<wire x1="374.65" y1="10.16" x2="382.27" y2="10.16" width="0.1524" layer="91"/>
+<pinref part="C72" gate="G$1" pin="1"/>
+<wire x1="374.65" y1="7.62" x2="374.65" y2="10.16" width="0.1524" layer="91"/>
+<junction x="374.65" y="10.16"/>
+<wire x1="334.01" y1="10.16" x2="374.65" y2="10.16" width="0.1524" layer="91"/>
+</segment>
+</net>

Commit message: All regulators done, pin out for sealed connector almost done, need outs for image sensor
Parts:
- removed JP8: (no value), pinhead:PINHD-1X2
- added C10, C11: 10uF, adafruit:C-USC0805
- added C18: 8200pF, adafruit:C-USC0805
- added C21, C9: 0.1uF, adafruit:C-USC0805
- added C24, C25, C26: 22uF, adafruit:C-USC0805
- added L3: 4.7uH, FormE:SRP6540
- added LED7: GREEN, FormE:LEDCHIPLED_0805
- added R10, R6, R8: 10K, adafruit:R-US_R0805
- added R5: 26.1K, adafruit:R-US_R0805
- added R9: 1K, adafruit:R-US_R0805
- added U3: TPS562219, FormE:TPS562219
- R24: value 54.9k -> 5.76K
Connections:
- removed net 12V_CURRENT_SENSE-: JP8.2, R15.2
- removed net N$54: C72.1, U21.IN
- removed net N$6: U2.PE0/AIN3/U7RX
- removed net N$7: U2.PB4/AIN10/CAN0RX/SSI2CLK/T1CCP0
- removed net N$8: U2.PD1/AIN6/I2C3SDA/SSI1FSS/SSI3FSS/WT2CCP1
- new net +1V2: C17.1, C19.1, C20.1, C23.1, L2.P$2, LED3.A, R24.2, U2.VDD, U2.VDD/1, U2.VDD/2, U2.VDD/3, U2.VDDA, U4.SPLIT/VIO
- new net +2V8: C24.1, C25.1, C26.1, L3.P$2, LED7.A, R5.2
- new net DAMPER_POS_OUT: H2.P23, U2.PA0/U0RX
- new net SS_5V2: C18.1, U3.SS
- new net STRAIN_GADGE_VOLTMETER_IN_0: H2.P19, U2.PE1/AIN2/U7TX, U2.PE3/AIN0
- new net STRAIN_GADGE_VOLTMETER_IN_1: H2.P18, U2.PE2/AIN1
- new net STRAIN_GAUGE_VOLTMETER_OUT: H2.P17, U2.PF0/C0O/CAN0RX/NMI/SSI1RX/TOCCPO/U1RTS
- new net SW_5V2: C21.2, L3.P$1, U3.SW
- new net VBST_5V2: C21.1, U3.VBST
- new net VFB_5V2: R5.1, R6.2, U3.VFB
- new net WHEEL_SPEED_OUT: R10.1, U2.PA4/SSI0RX
- net +12V: now also H2.P1, H2.P16, H2.P9, R10.2, R15.2; no longer JP8.1
- net +3V3: now also H2.P7, H2.P8; no longer C23.1, U2.VDD, U2.VDD/1, U2.VDD/2, U2.VDD/3, U2.VDDA, U4.SPLIT/VIO
- net +5V: no longer C17.1, C19.1, C20.1, L2.P$2, LED3.A, R24.2
- net GND: now also C10.2, C11.2, C18.2, C24.2, C25.2, C26.2, C9.2, H2.P2, H2.P3, H2.P4, H2.P5, H2.P6, R6.1, R9.1, U3.GND
- net N$3: now also LED7.C, R9.2; no longer U2.PE3/AIN0
- net N$4: now also R8.2, U3.EN; no longer U2.PE2/AIN1
- net N$5: now also H2.P10; no longer U2.PE1/AIN2/U7TX
- net PROGRAMMING_CAN_N: now also H2.P22
- net PROGRAMMING_CAN_P: now also H2.P21
- net PROGRAMMING_CAN_RX: now also U2.PB4/AIN10/CAN0RX/SSI2CLK/T1CCP0; no longer U2.PF0/C0O/CAN0RX/NMI/SSI1RX/TOCCPO/U1RTS
- net VCC: now also C10.1, C11.1, C72.1, C9.1, H2.P20, R8.1, U21.IN, U3.VIN
Other:
- note added: "+12V to Damper Pos, Strain Gauge, and Wheel Speed Sensor"
- note added: "+1V2 and +2V8 to Image Sensor"
- note added: "<-- R1 <-- R2"
- note added: "General IO for CAN? PWM?"
- note added: "Input clock 25-MHz nominal, CMOS IO Voltage Levels Video data interface Video over SPI Control port CCI (I2C-like), CMOS IO Voltage Levels"
- note added: "Need back in for CAN?"
- note added: "To enable differential sampling, software must set the Dn bit in the ADCSSCTL0n register in a step's configuration nibble. TM4C1231C3PM 774"
- note added: "User-selectable 14-bit, 8-bit (AGC applied), or 24-bit RGB (AGC and colorization applied)?????????????????????????????"
- note added: "VCC from low volt battery, between 12.8V and 16.8V"
- note added: "Vout = .765*(1+(R1/R2)) VOUT | R1 -------|--------- 5.0V | 54.9K 3.3V | 33.2K 2.8V | 26.1K 1.8V | 13.7K 1.2V | 5.76K"
- note removed: "VOUT | R1 -------|--------- 5.0V | 54.9K 3.3V | 33.2K 1.8V | 13.7K 1.2V | 5.76K"
- moved on the sheet: C1, C12, C13, C14, C15, C16, C17, C19, C2, C20, C3, C4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

Commit message: About to delete 1V2 and 2V8 Regulators because switching Image sensor
Parts:
- removed H2: 776228-4, FormE:776228-4
- added H1: 1-776231-1, FormE:1-776231-1
Connections:
- removed net N$5: H2.P10
- net +12V: now also H1.1, H1.21, H1.28; no longer H2.P1, H2.P16, H2.P9
- net +3V3: now also H1.7, H1.8; no longer H2.P7, H2.P8
- net DAMPER_POS_OUT: now also H1.35; no longer H2.P23
- net GND: now also H1.2, H1.3, H1.4, H1.5, H1.6; no longer H2.P2, H2.P3, H2.P4, H2.P5, H2.P6
- net PROGRAMMING_CAN_N: now also H1.34; no longer H2.P22
- net PROGRAMMING_CAN_P: now also H1.33; no longer H2.P21
- net STRAIN_GADGE_VOLTMETER_IN_0: now also H1.31; no longer H2.P19
- net STRAIN_GADGE_VOLTMETER_IN_1: now also H1.30; no longer H2.P18
- net STRAIN_GAUGE_VOLTMETER_OUT: now also H1.29; no longer H2.P17
- net VCC: now also H1.32; no longer H2.P20
- net WHEEL_SPEED_OUT: now also H1.22
Other:
- note removed: "Input clock 25-MHz nominal, CMOS IO Voltage Levels Video data interface Video over SPI Control port CCI (I2C-like), CMOS IO Voltage Levels"
- note removed: "User-selectable 14-bit, 8-bit (AGC applied), or 24-bit RGB (AGC and colorization applied)?????????????????????????????"

Commit message: Everything done exept for scary LEDs
Parts:
- removed C21: 0.1uF, adafruit:C-USC0805
- removed C24, C25, C26: 22uF, adafruit:C-USC0805
- removed L3: 4.7uH, FormE:SRP6540
- removed LED7: GREEN, FormE:LEDCHIPLED_0805
- removed R24: 5.76K, adafruit:R-US_R0805
- removed R25, R26: 10K, adafruit:R-US_R0805
- removed R27: 1K, adafruit:R-US_R0805
- removed U10: TPS562219, FormE:TPS562219
- C12: value 0.1uF -> 8200pF; PARTNO GRM21BR71E104KA01L -> C0805C822K5RACTU
- C13: value 10uF -> 0.1uF; PARTNO GRM21BR61E106KA73L -> GRM21BR71E104KA01L
- C14: value 10uF -> 22uF; PARTNO GRM21BR61E106KA73L -> C2012JB1E226M125AC
- C15: value 8200pF -> 22uF; PARTNO C0805C822K5RACTU -> C2012JB1E226M125AC
- C16: value 0.1uF -> 22uF; PARTNO GRM21BR71E104KA01L -> C2012JB1E226M125AC
- C17, C19, C20: value 22uF -> 0.1uF; device adafruit:C-USC0805 -> rcl:C-USC0805; PARTNO C2012JB1E226M125AC -> GRM21BR71H104KA01L
- C18: value 8200pF -> 0.1uF; device adafruit:C-USC0805 -> rcl:C-USC0805; PARTNO C0805C822K5RACTU -> GRM21BR71H104KA01L
- R5: value 26.1K -> 33.2K
Connections:
- removed net +1V2: C17.1, C19.1, C20.1, C23.1, L2.P$2, LED3.A, R24.2, U2.VDD, U2.VDD/1, U2.VDD/2, U2.VDD/3, U2.VDDA, U4.SPLIT/VIO
- removed net +2V8: C24.1, C25.1, C26.1, L3.P$2, LED7.A, R5.2
- removed net N$1001: R26.2, U10.EN
- removed net N$28: LED3.C, R27.2
- removed net SS_5V: C15.1, U10.SS
- removed net SW_5V: C16.2, L2.P$1, U10.SW
- removed net VBST_5V: C16.1, U10.VBST
- removed net VFB_5V: R24.1, R25.2, U10.VFB
- new net IR_SENSOR_1_ANALOG_OUT: H1.28, U2.PD0/AIN7/I2C3SCL/SSI1CLK/SSI3CLK/WT2CCP0
- new net IR_SENSOR_1_DIGITAL_IN: H1.12, U2.PB0/T2CCP0/U1RX
- new net IR_SENSOR_1_DIGITAL_OUT: H1.15, U2.PC3/SWO/T5CCP1/TDO
- new net IR_SENSOR_2_ANALOG_OUT: H1.27, U2.PD1/AIN6/I2C3SDA/SSI1FSS/SSI3FSS/WT2CCP1
- new net IR_SENSOR_2_DIGITAL_IN: H1.11, U2.PC2/T5CCP0/TDI
- new net IR_SENSOR_2_DIGITAL_OUT: H1.14, U2.PB3/I2C0SDA/T3CCP1
- new net IR_SENSOR_3_ANALOG_OUT: H1.26, U2.PD2/AIN5/SSI1RX/SSI3RX/WT3CCP0
- new net IR_SENSOR_3_DIGITAL_IN: H1.10, U2.PC1/SWDIO/T4CCP1/TMS
- new net IR_SENSOR_3_DIGITAL_OUT: H1.13, U2.PB2/I2C0SCL/T3CCP0
- net +12V: now also H1.2, H1.3, H1.4, H1.5, H1.6; no longer H1.21, H1.28
- net +3V3: now also C17.1, C18.1, C19.1, C20.1, C23.1, U2.VDD, U2.VDD/1, U2.VDD/2, U2.VDD/3, U2.VDDA, U4.SPLIT/VIO; no longer H1.7, H1.8
- net +5V: now also C14.1, C15.1, C16.1, L2.P$2, LED3.A, R5.2
- net DAMPER_POS_OUT: now also H1.25; no longer H1.35
- net GND: now also C16.2, H1.17, H1.18, H1.19, H1.20; no longer C13.2, C24.2, C25.2, C26.2, H1.2, H1.3, H1.4, H1.5, H1.6, R25.1, R27.1, U10.GND
- net N$3: now also LED3.C; no longer LED7.C
- net PROGRAMMING_CAN_N: now also H1.35; no longer H1.34
- net PROGRAMMING_CAN_P: now also H1.34; no longer H1.33
- net SS_5V2: now also C12.1; no longer C18.1
- net STRAIN_GADGE_VOLTMETER_IN_0: no longer U2.PE1/AIN2/U7TX
- net STRAIN_GAUGE_VOLTMETER_OUT: no longer U2.PF0/C0O/CAN0RX/NMI/SSI1RX/TOCCPO/U1RTS
- net SW_5V2: now also C13.2, L2.P$1; no longer C21.2, L3.P$1
- net VBST_5V2: now also C13.1; no longer C21.1
- net VCC: no longer C12.1, C13.1, C14.1, R26.1, U10.VIN
- net WHEEL_SPEED_OUT: now also H1.24; no longer H1.22
Other:
- note removed: "+12V to Damper Pos, Strain Gauge, and Wheel Speed Sensor"
- note removed: "+1V2 and +2V8 to Image Sensor"
- moved on the sheet: C10, C11, C12, C13, C14, C15, C16, C17, C18, C19, C20, C27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

Commit message: Done  (1st)
Parts:
- added C21: 0.1uF, rcl:C-USC0805
- added LED10, LED11, LED12, LED13, LED14, LED15, LED16, LED17, LED18, LED7, LED8, LED9: APA102C, FormE:APA102C
- U2: value (none) -> TM4C1231C3PM
Connections:
- removed net N$17: LED1.DI
- removed net N$18: LED1.CI
- removed net STRAIN_GAUGE_VOLTMETER_OUT: H1.29
- new net N$12: LED4.CO, LED7.CI
- new net N$13: LED4.DO, LED7.DI
- new net N$14: LED10.DO, LED11.DI
- new net N$19: LED11.DO, LED12.DI
- new net N$20: LED11.CO, LED12.CI
- new net N$21: LED10.CO, LED11.CI
- new net N$22: LED10.DI, LED9.DO
- new net N$23: LED10.CI, LED9.CO
- new net N$24: LED13.DO, LED14.DI
- new net N$25: LED14.DO, LED15.DI
- new net N$26: LED14.CO, LED15.CI
- new net N$27: LED13.CO, LED14.CI
- new net N$28: LED12.DO, LED13.DI
- new net N$29: LED12.CO, LED13.CI
- new net N$30: LED16.DO, LED17.DI
- new net N$31: LED17.DO, LED18.DI
- new net N$32: LED17.CO, LED18.CI
- new net N$33: LED16.CO, LED17.CI
- new net N$34: LED15.CO, LED16.CI
- new net N$35: LED15.DO, LED16.DI
- new net N$5: LED7.DO, LED8.DI
- new net N$6: LED8.DO, LED9.DI
- new net N$7: LED8.CO, LED9.CI
- new net N$8: LED7.CO, LED8.CI
- net +3V3: now also C21.1
- net +5V: now also LED10.+5V, LED11.+5V, LED12.+5V, LED13.+5V, LED14.+5V, LED15.+5V, LED16.+5V, LED17.+5V, LED18.+5V, LED7.+5V, LED8.+5V, LED9.+5V
- net GND: now also C21.2, H1.21, H1.22, H1.23, LED10.GND, LED11.GND, LED12.GND, LED13.GND, LED14.GND, LED15.GND, LED16.GND, LED17.GND, LED18.GND, LED7.GND, LED8.GND, LED9.GND; no longer H1.17, H1.18, H1.19
- net IR_SENSOR_1_ANALOG_OUT: now also H1.30; no longer H1.28
- net IR_SENSOR_1_DIGITAL_IN: now also H1.19, U2.PC0/SWCLK/T4CCP0/TCK; no longer H1.12, U2.PB0/T2CCP0/U1RX
- net IR_SENSOR_2_ANALOG_OUT: now also H1.29; no longer H1.27
- net IR_SENSOR_2_DIGITAL_IN: now also H1.18, U2.PC1/SWDIO/T4CCP1/TMS; no longer H1.11, U2.PC2/T5CCP0/TDI
- net IR_SENSOR_3_ANALOG_OUT: now also H1.28; no longer H1.26
- net IR_SENSOR_3_DIGITAL_IN: now also H1.17, U2.PC2/T5CCP0/TDI; no longer H1.10, U2.PC1/SWDIO/T4CCP1/TMS
- net SPI_SCARY_LED_CLOCK: now also LED1.CI
- net SPI_SCARY_LED_TRANSMIT: now also LED1.DI
- net STRAIN_GADGE_VOLTMETER_IN_0: now also H1.27; no longer H1.31
- net STRAIN_GADGE_VOLTMETER_IN_1: now also H1.26; no longer H1.30
Other:
- moved on the sheet: LED1, LED2, LED4
