File: Artemis Corner Board V2 FR.sch (EAGLE design)
At the start: 91 parts, among them Q1 BSS138, U1 OPA365AIDBVR, U2 ADS1232IPWR, U3 MCP2562, U4 TM4C123GH6PMI, U5 MCP2562, U6 LM3671MF-3.3/NOPB, U8 TPS562219, U9 FT232RL, Y1 16MHz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

Commit message: Added a few notes, about to start on new Corner DAQ Board
Other:
- note added: "IR SENSOR http://www.omega.com/pptst/OS137.html - 9m dist?"
- note added: "NOPE ---->"
- note added: "Strain Gauge: Micro-Measurements MMF003129 (125UN series) http://www.digikey.com/product-detail/en/CEA-06-125UN-350/1033-1004-ND/2503695 -Needs own board, use precision 350 resistors for wheatstone bridge, -use dual strain gadge setup to minimize effect of temperature -maybe 3 wire connection? -need very accurate Vin so use V regulator to go from Vbatt --> 6V or 7V then use a linear regulator to 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"
- note removed: "Strain Gauge: Micro-Measurements MMF003129 (125UN series) http://www.digikey.com/product-detail/en/CEA-06-125UN-350/1033-1004-ND/2503695 Requires 3 additional 350-ohm precision resistors to form a wheatstone bridge"
Changed lines of the file:
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@@
 <?xml version="1.0" encoding="utf-8"?>
 <!DOCTYPE eagle SYSTEM "eagle.dtd">
-<eagle version="7.3.0">
+<eagle version="7.5.0">
 <drawing>
 <settings>
@@
 HIGH: use AIN2
 LOW: use AIN1</text>
-<text x="-746.76" y="160.02" size="1.778" layer="97">Hall Effect Sensor:
+<text x="-746.76" y="144.78" size="1.778" layer="97">Hall Effect Sensor:
 Texense RS-M10 WS
 http://www.sens4speed.com/en/products/wheel-speed/rs-m10ws_3.html</text>
-<text x="-746.76" y="147.32" size="1.778" layer="97">Shock Potentiometer:
+<text x="-746.76" y="134.62" size="1.778" layer="97">Shock Potentiometer:
 Texense RSL 75mm
 http://www.sens4speed.com/en/products/potentiometers/rsl-75mm_14.html</text>
-<text x="-746.76" y="134.62" size="1.778" layer="97">IR Camera:
+<text x="-746.76" y="177.8" size="1.778" layer="97">IR Camera:
 Flir Lepton 500-0659-01
 http://www.digikey.com/product-detail/en/500-0659-01/500-0659-01-ND/5215153</text>
-<text x="-746.76" y="111.76" size="1.778" layer="97">Strain Gauge:
+<text x="-746.76" y="81.28" size="1.778" layer="97">Strain Gauge:
 Micro-Measurements MMF003129
 (125UN series)
 http://www.digikey.com/product-detail/en/CEA-06-125UN-350/1033-1004-ND/2503695
-  Requires 3 additional
-  350-ohm precision resistors
-  to form a wheatstone bridge</text>
+-Needs own board, use precision 350 resistors
+for wheatstone bridge,
+-use dual strain gadge setup to minimize
+effect of temperature
+-maybe 3 wire connection?
+-need very accurate Vin
+so use V regulator to go from Vbatt --&gt; 6V or 7V
+then use a linear regulator to get down to 5V
+-The people whose ideas im stealing:
+http://edge.rit.edu/edge/P05109/public
+/Files/PDR.pdf
+-The part they use:  AD8230</text>
 <text x="-495.3" y="195.58" size="1.27" layer="97" rot="MR0">GLV battery VCC</text>
 <text x="-495.3" y="172.72" size="1.27" layer="97" rot="MR0">GLV battery GND</text>
@@
 <text x="-205.74" y="139.7" size="1.778" layer="97">NC</text>
 <text x="810.26" y="170.18" size="1.778" layer="97">74479775222</text>
+<text x="-746.76" y="154.94" size="1.778" layer="95">IR SENSOR
+http://www.omega.com/pptst/OS137.html   - 9m dist?</text>
+<text x="-762" y="180.34" size="1.778" layer="91">NOPE ----&gt;</text>
 </plain>
 <instances>
